Commit message: how to sim

File: assembly_sim/urdf/sim_robot.urdf.xacro (robot description, xacro)
@@ -73,5 +73,5 @@
         <parent link="table" />
         <child link = "robot2_base_link" />
-        <origin xyz="1.0 0.0 0.01" rpy="0.0 0.0 0.0" />
+        <origin xyz="0.75 0.0 0.01" rpy="0.0 0.0 0.0" />
     </joint>
 </robot>
